Commit message: MZ04 simulation in moveit

File: mz04/urdf/mz04.urdf (robot description, URDF)
Before this commit: robot mz04, 8 links, 7 joints
Joints:
- joint J1: limit lower=-2.97 upper=2.97 effort=100 velocity=1 -> lower=-2.97 upper=2.97 effort=100 velocity=8.38
- joint J2: axis 0 0 1 -> 0 0 -1; limit lower=-2.53 upper=1.57 effort=100 velocity=1 -> lower=-2.53 upper=1.57 effort=100 velocity=8.03
- joint J3: limit lower=-2.18 upper=4.88 effort=100 velocity=1 -> lower=-1.22 upper=3.31 effort=100 velocity=9.08
- joint J4: limit lower=-3.32 upper=3.32 effort=100 velocity=1 -> lower=-3.32 upper=3.32 effort=100 velocity=9.77
- joint J5: limit lower=-2.09 upper=2.09 effort=100 velocity=1 -> lower=-2.09 upper=2.09 effort=100 velocity=9.77
- joint J6: limit lower=-6.28 upper=6.28 effort=100 velocity=1 -> lower=-6.28 upper=6.28 effort=100 velocity=15.7
